Commit message: Migrate quadruped_robot V1.1 to htdw-4438 V1.2
Renamed and reorganized the quadruped_robot V1.1 hardware package to htdw-4438 V1.2, including all configuration, launch, mesh, and URDF files. Added new mesh files for FR_foot and RL_foot, and included export.log and URDF.SLDASM.csv for the new version. Removed corresponding files from the old package.

File: 1.Hardware/htdw-4438 V1.2/urdf/URDF.SLDASM.urdf (robot description, URDF)
Before this commit: robot htdw_4438, 17 links, 16 joints
Links:
- link base_link: mass 2.6821 -> 2.68214792; geometry collision mesh filename=package://htdw_4438/meshes/base_link.STL; visual mesh filename=package://htdw_4438/meshes/base_link.STL
- link fl_calf: mass 0.0403 -> 0.04033111; geometry collision mesh filename=package://htdw_4438/meshes/FL_calf.STL; visual mesh filename=package://htdw_4438/meshes/FL_calf.STL
- link fl_foot: mass 0.0066 -> 0.00657865; geometry collision mesh filename=package://htdw_4438/meshes/FL_foot.STL; visual mesh filename=package://htdw_4438/meshes/FL_foot.STL
- link fl_hip: mass 0.2924 -> 0.29235822; geometry collision mesh filename=package://htdw_4438/meshes/FL_hip.STL; visual mesh filename=package://htdw_4438/meshes/FL_hip.STL
- link fl_thigh: mass 0.4104 -> 0.41040818; geometry collision mesh filename=package://htdw_4438/meshes/FL_thigh.STL; visual mesh filename=package://htdw_4438/meshes/FL_thigh.STL
- link fr_calf: mass 0.0403 -> 0.04033111; geometry collision mesh filename=package://htdw_4438/meshes/FR_calf.STL; visual mesh filename=package://htdw_4438/meshes/FR_calf.STL
- link fr_foot: mass 0.0066 -> 0.00657865; geometry collision mesh filename=package://htdw_4438/meshes/FR_foot.STL; visual mesh filename=package://htdw_4438/meshes/FR_foot.STL
- link fr_hip: mass 0.2924 -> 0.29235822; geometry collision mesh filename=package://htdw_4438/meshes/FR_hip.STL; visual mesh filename=package://htdw_4438/meshes/FR_hip.STL
- link fr_thigh: mass 0.4104 -> 0.41040818; geometry collision mesh filename=package://htdw_4438/meshes/FR_thigh.STL; visual mesh filename=package://htdw_4438/meshes/FR_thigh.STL
- link rl_calf: mass 0.0403 -> 0.04033111; geometry collision mesh filename=package://htdw_4438/meshes/RL_calf.STL; visual mesh filename=package://htdw_4438/meshes/RL_calf.STL
- link rl_foot: mass 0.0066 -> 0.00657865; geometry collision mesh filename=package://htdw_4438/meshes/RL_foot.STL; visual mesh filename=package://htdw_4438/meshes/RL_foot.STL
- link rl_hip: mass 0.2924 -> 0.29235822; geometry collision mesh filename=package://htdw_4438/meshes/RL_hip.STL; visual mesh filename=package://htdw_4438/meshes/RL_hip.STL
- link rl_thigh: mass 0.4104 -> 0.41040818; geometry collision mesh filename=package://htdw_4438/meshes/RL_thigh.STL; visual mesh filename=package://htdw_4438/meshes/RL_thigh.STL
- link rr_calf: mass 0.0403 -> 0.04033111; geometry collision mesh filename=package://htdw_4438/meshes/RR_calf.STL; visual mesh filename=package://htdw_4438/meshes/RR_calf.STL
- link rr_foot: mass 0.0066 -> 0.00657865; geometry collision mesh filename=package://htdw_4438/meshes/RR_foot.STL; visual mesh filename=package://htdw_4438/meshes/RR_foot.STL
- link rr_hip: mass 0.2924 -> 0.29235822; geometry collision mesh filename=package://htdw_4438/meshes/RR_hip.STL; visual mesh filename=package://htdw_4438/meshes/RR_hip.STL
- link rr_thigh: mass 0.4104 -> 0.41040818; geometry collision mesh filename=package://htdw_4438/meshes/RR_thigh.STL; visual mesh filename=package://htdw_4438/meshes/RR_thigh.STL

Commit message: Update

File: 1.Hardware/htdw-4438 V1.2/urdf/URDF.SLDASM.urdf (robot description, URDF)
Before this commit: robot htdw_4438, 17 links, 16 joints
Joints:
- joint fl_calf_joint: limit lower=-0.5236 upper=0.5236 effort=2 velocity=4.7124 -> lower=-2.5 upper=-1.5 effort=10 velocity=9.95
- joint fl_hip_joint: axis -1 0 0 -> 1 0 0; limit lower=-0.5236 upper=0.5236 effort=2 velocity=4.7124 -> lower=-0.3 upper=0.6 effort=10 velocity=9.95
- joint fl_thigh_joint: limit lower=-0.5236 upper=0.5236 effort=2 velocity=4.7124 -> lower=0.2 upper=1.5 effort=10 velocity=9.95
- joint fr_calf_joint: limit lower=-0.5236 upper=0.5236 effort=2 velocity=4.7124 -> lower=-2.5 upper=-1.5 effort=10 velocity=9.95
- joint fr_hip_joint: limit lower=-0.5236 upper=0.5236 effort=2 velocity=4.7124 -> lower=-0.6 upper=0.3 effort=10 velocity=9.95
- joint fr_thigh_joint: axis 0 -1 0 -> 0 1 0; limit lower=-0.5236 upper=0.5236 effort=2 velocity=4.7124 -> lower=0.2 upper=1.5 effort=10 velocity=9.95
- joint rl_calf_joint: limit lower=-0.5236 upper=0.5236 effort=2 velocity=4.7124 -> lower=-2.5 upper=-1.5 effort=10 velocity=9.95
- joint rl_hip_joint: axis -1 0 0 -> 1 0 0; limit lower=-0.5236 upper=0.5236 effort=2 velocity=4.7124 -> lower=-0.3 upper=0.6 effort=10 velocity=9.95
- joint rl_thigh_joint: limit lower=-0.5236 upper=0.5236 effort=2 velocity=4.7124 -> lower=0.2 upper=1.5 effort=10 velocity=9.95
- joint rr_calf_joint: limit lower=-0.5236 upper=0.5236 effort=2 velocity=4.7124 -> lower=-2.5 upper=-1.5 effort=10 velocity=9.95
- joint rr_hip_joint: limit lower=-0.5236 upper=0.5236 effort=2 velocity=4.7124 -> lower=-0.6 upper=0.3 effort=10 velocity=9.95
- joint rr_thigh_joint: axis 0 -1 0 -> 0 1 0; limit lower=-0.5236 upper=0.5236 effort=2 velocity=4.7124 -> lower=0.2 upper=1.5 effort=10 velocity=9.95
