Commit message: 修改URDF版本

File: 1.Hardware/htdw_4438/urdf/htdw_4438.urdf (robot description, URDF)
Before this commit: robot htdw_4438, 17 links, 16 joints
Links:
- link base_link: geometry collision box size=0.18 0.0935 0.138; visual mesh filename=../meshes/base_link.STL
- link fl_calf: geometry collision cylinder length=0.12 radius=0.01; visual mesh filename=../meshes/FL_calf.STL
- link fl_foot: geometry collision sphere radius=0.015; visual mesh filename=../meshes/FL_foot.STL
- link fl_hip: geometry collision box size=0.06 0.047 0.062; visual mesh filename=../meshes/FL_hip.STL
- link fl_thigh: geometry collision box size=0.05 0.025 0.12; visual mesh filename=../meshes/FL_thigh.STL
- link fr_calf: geometry collision cylinder length=0.12 radius=0.01; visual mesh filename=../meshes/FR_calf.STL
- link fr_foot: geometry collision sphere radius=0.015; visual mesh filename=../meshes/FR_foot.STL
- link fr_hip: geometry collision box size=0.06 0.047 0.062; visual mesh filename=../meshes/FR_hip.STL
- link fr_thigh: geometry collision box size=0.05 0.025 0.12; visual mesh filename=../meshes/FR_thigh.STL
- link rl_calf: geometry collision cylinder length=0.12 radius=0.01; visual mesh filename=../meshes/RL_calf.STL
- link rl_foot: geometry collision sphere radius=0.015; visual mesh filename=../meshes/RL_foot.STL
- link rl_hip: geometry collision box size=0.06 0.047 0.062; visual mesh filename=../meshes/RL_hip.STL
- link rl_thigh: geometry collision box size=0.05 0.025 0.12; visual mesh filename=../meshes/RL_thigh.STL
- link rr_calf: geometry collision cylinder length=0.12 radius=0.01; visual mesh filename=../meshes/RR_calf.STL
- link rr_foot: geometry collision sphere radius=0.015; visual mesh filename=../meshes/RR_foot.STL
- link rr_hip: geometry collision box size=0.06 0.047 0.062; visual mesh filename=../meshes/RR_hip.STL
- link rr_thigh: geometry collision box size=0.05 0.025 0.12; visual mesh filename=../meshes/RR_thigh.STL
Joints:
- joint fl_calf_joint: limit lower=-2.5 upper=-1.5 effort=10 velocity=9.95 -> lower=-2.5 upper=-1.2 effort=10 velocity=9.95
- joint fl_hip_joint: limit lower=-0.3 upper=0.6 effort=10 velocity=9.95 -> lower=-0.9 upper=0.9 effort=10 velocity=9.95
- joint fl_thigh_joint: limit lower=0.2 upper=1.5 effort=10 velocity=9.95 -> lower=-1.5 upper=3.5 effort=10 velocity=9.95
- joint fr_calf_joint: limit lower=-2.5 upper=-1.5 effort=10 velocity=9.95 -> lower=-2.5 upper=-1.2 effort=10 velocity=9.95
- joint fr_hip_joint: limit lower=-0.6 upper=0.3 effort=10 velocity=9.95 -> lower=-0.9 upper=0.9 effort=10 velocity=9.95
- joint fr_thigh_joint: limit lower=0.2 upper=1.5 effort=10 velocity=9.95 -> lower=-1.5 upper=3.5 effort=10 velocity=9.95
- joint rl_calf_joint: limit lower=-2.5 upper=-1.5 effort=10 velocity=9.95 -> lower=-2.5 upper=-1.2 effort=10 velocity=9.95
- joint rl_hip_joint: limit lower=-0.3 upper=0.6 effort=10 velocity=9.95 -> lower=-0.9 upper=0.9 effort=10 velocity=9.95
- joint rl_thigh_joint: limit lower=0.2 upper=1.5 effort=10 velocity=9.95 -> lower=-1.5 upper=3.5 effort=10 velocity=9.95
- joint rr_calf_joint: limit lower=-2.5 upper=-1.5 effort=10 velocity=9.95 -> lower=-2.5 upper=-1.2 effort=10 velocity=9.95
- joint rr_hip_joint: limit lower=-0.6 upper=0.3 effort=10 velocity=9.95 -> lower=-0.9 upper=0.9 effort=10 velocity=9.95
- joint rr_thigh_joint: limit lower=0.2 upper=1.5 effort=10 velocity=9.95 -> lower=-1.5 upper=3.5 effort=10 velocity=9.95
